Commit message: update after RoboCup '16 in Leipzig, Germany

File: mas_industrial_robotics/mir_robots/mir_hardware_config/youbot-brsu-4/urdf/robot.urdf.xacro (robot description, xacro)
@@ -6,14 +6,14 @@
        name="youbot" >
   <!-- The following included files set up definitions of parts of the robot body -->
-  <!-- misc common stuff? -->
+  <!-- misc common stuff -->
   <xacro:include filename="$(find youbot_description)/urdf/common.xacro" />
-  <!-- youbot base -->
+  <xacro:include filename="$(find mcr_description)/urdf/materials.urdf.xacro" />
+  <!-- youbot base and rear platform -->
   <xacro:include filename="$(find youbot_description)/urdf/youbot_base/base.urdf.xacro" />
-  <!-- youbot plate -->
-  <xacro:include filename="$(find youbot_description)/urdf/youbot_plate/plate.urdf.xacro" />
-  <!-- youbot arm -->
+  <xacro:include filename="$(find mir_description)/urdf/misc/rear_platform_v2.urdf.xacro" />
+  <!-- youbot arm and gripper-->
   <xacro:include filename="$(find youbot_description)/urdf/youbot_arm/arm.urdf.xacro"/>
-  <!-- youbot gripper -->
-  <xacro:include filename="$(find youbot_description)/urdf/youbot_gripper/gripper.urdf.xacro" />
+  <xacro:include filename="$(find mir_description)/urdf/misc/adapter_plate.urdf.xacro" />
+  <xacro:include filename="$(find mir_description)/urdf/grippers/dynamixel/v2/dynamixel_gripper.urdf.xacro" />
   <!-- controller manager -->
   <xacro:include filename="$(find youbot_description)/controller/ros_controller.urdf.xacro" />
@@ -22,56 +22,38 @@
   <!-- sensors -->
   <xacro:include filename="$(find youbot_description)/urdf/sensors/hokuyo_urg04_laser.urdf.xacro"/>
+  <xacro:include filename="$(find mir_description)/urdf/sensor_mounts/intel_f200_camera_mount.urdf.xacro"/>
+  <xacro:include filename="$(find mcr_description)/urdf/sensors/intel_realsense_f200_camera.urdf.xacro"/>
   <!-- Now we can start using the macros included above to define the actual youbot -->
-  <!-- The first use of a macro.  This one was defined in base.urdf.xacro above.
-       A macro like this will expand to a set of link and joint definitions, and to additional
-       Gazebo-related extensions (sensor plugins, etc).  The macro takes an argument, name,
-       that equals "base", and uses it to generate names for its component links and joints
-       (e.g., base_link).  The included origin block is also an argument to the macro.  By convention,
-       the origin block defines where the component is w.r.t its parent (in this case the parent
-       is the world frame). For more, see http://www.ros.org/wiki/xacro -->
-  <!-- foot for arm-->
+  <!-- standard youBot configuration -->
   <xacro:youbot_base name="base"/>
-  <!-- BRSU SPECIFIC STUFF -->
-  <xacro:include filename="$(find mcr_description)/urdf/materials.urdf.xacro" />
-  <xacro:include filename="$(find mir_description)/urdf/misc/cam3d_tower.urdf.xacro"/>
-  <xacro:include filename="$(find mcr_description)/urdf/sensors/asus_xtion_camera.urdf.xacro"/>
-  <xacro:include filename="$(find mcr_description)/urdf/mounts/microsoft_lifecam_1080_mount.urdf.xacro"/>
-  <xacro:include filename="$(find mir_description)/urdf/misc/rear_platform.urdf.xacro" />
-  <xacro:include filename="$(find mir_description)/urdf/misc/adapter_plate.urdf.xacro" />
-  <xacro:include filename="$(find mir_description)/urdf/grippers/festo_gripper.urdf.xacro" />
   <!-- Rear Platform -->
-  <xacro:rear_platform name="rear_platform" parent="base_link">
-    <origin xyz="-0.005 -0.175 0.051" rpy="0 0 0" />
-  </xacro:rear_platform>
+  <xacro:rear_platform_v2 name="rear_platform" parent="base_link">
+    <origin xyz="0.12 -0.175 ${0.021 + 0.0062 + 0.025 + 0.012}" rpy="0 0 0" />  <!-- ${alignment with base top + nut height + spacer height + slide height } -->
+  </xacro:rear_platform_v2>
   <!-- Arm Plate moving arm 8cm foward and 45 degree rotation -->
   <xacro:adapter_plate name="adapter_plate" parent="base_link" arm_angle="${-M_PI / 4}">
-    <origin xyz="${0.159+0.08} 0 0.051" rpy="0 0 0" />
+    <origin xyz="${0.159+0.08} 0 ${0.021 + 0.025 + 0.025}" rpy="0 0 0" />    <!-- ${alignment with base top + spacer height + spacer height } -->
   </xacro:adapter_plate>
   <xacro:youbot_arm name="arm" parent="adapter_plate_arm_root_link">
     <origin xyz="-0.022 0.0 0.037" rpy="0 0 0" />
   </xacro:youbot_arm>
-  <!-- Festo Gripper -->
-  <xacro:festo_gripper name="gripper" parent="arm_link_5">
-    <origin xyz="0 0 0" rpy="0 0 0" />
-  </xacro:festo_gripper>
   <!-- base laser front -->
   <xacro:hokuyo_urg04_laser name="base_laser_front" parent="base" ros_topic="scan_front" update_rate="10" min_angle="-1.57" max_angle="1.57">
-    <origin xyz="0.3 0 -0.03" rpy="0 0 0"/>
+    <origin xyz="0.3 0 -0.035" rpy="${M_PI} 0 0"/>
   </xacro:hokuyo_urg04_laser>
   <!-- base laser rear -->
   <xacro:hokuyo_urg04_laser name="base_laser_rear" parent="base" ros_topic="scan_rear" update_rate="10" min_angle="-1.57" max_angle="1.57" >
-     <origin xyz="-0.3 0 -0.03" rpy="0 0 ${M_PI}" />
+     <origin xyz="-0.3 0.0 -0.035" rpy="${M_PI} 0 ${M_PI}" />
   </xacro:hokuyo_urg04_laser>
-  <!-- camera tower -->
-  <xacro:cam3d_tower name="camera_tower" parent="rear_platform_link">
-    <origin xyz="-0.227 0.165 0.023" rpy="0 0 0" />
-  </xacro:cam3d_tower>
-  <!-- 3D camera on tower -->
-  <xacro:asus_xtion_camera name="tower_cam3d" parent="camera_tower_link" tilt="0.5">
-    <origin xyz="0.015 0 0.47" rpy="0 0 0" />
-  </xacro:asus_xtion_camera>
-  <!-- Arm POV Mount -->
-  <xacro:microsoft_lifecam_1080_mount name="microsoft_lifecam_1080_mount" parent="arm_link_5">
-    <origin xyz="-0.035 0.0 -0.025" rpy="0 0 3.14159265" />
-  </xacro:microsoft_lifecam_1080_mount>
+  <xacro:dynamixel_gripper_v2 name="gripper" parent="arm_link_5">
+    <origin xyz="0.003 0 0.0052" rpy="0 0 0" />
+  </xacro:dynamixel_gripper_v2>
+  <!-- camera mount for Intel RealSense F200 -->
+  <xacro:intel_f200_camera_mount name="camera_mount" parent="gripper_motor_mount_link">
+    <origin xyz="-0.00375 -0.0007 0.012" rpy="-0.05 -0.04 0" />
+  </xacro:intel_f200_camera_mount>
+  <!-- 3D camera on arm -->
+  <xacro:intel_realsense_f200_camera name="arm_cam3d" parent="camera_mount_link">
+    <origin xyz="-0.0405 -0.008 0.025" rpy="-0.2 -${M_PI/2} 0" />
+  </xacro:intel_realsense_f200_camera>
 </robot>
